Commit message: update for gazebo

File: magician_description/urdf/magician.urdf.xacro (robot description, xacro)
@@ -4,5 +4,8 @@
      For more information, please see http://wiki.ros.org/sw_urdf_exporter -->
 <robot
-  name="magician">
+  name="magician" xmlns:xacro="http://www.ros.org/wiki/xacro">
+  <xacro:include filename="$(find magician_description)/urdf/materials.xacro" />
+  <xacro:include filename="$(find magician_description)/urdf/magician.gazebo" />
+  <xacro:include filename="$(find magician_description)/urdf/magician_transmission.xacro" />
   <link name="world"/>
   <link name="magician_origin"/>
@@ -19,6 +22,4 @@
     <axis
       xyz="0 0 0" />
-    <safety_controller
-      k_velocity="0" />
   </joint>
   <link
@@ -74,6 +75,4 @@
     <axis
       xyz="0 0 0" />
-    <safety_controller
-      k_velocity="0" />
   </joint>
   <link
@@ -132,8 +131,6 @@
       lower="-2.1816"
       upper="2.1816"
-      effort="0"
-      velocity="0" />
-    <safety_controller
-      k_velocity="0" />
+      effort="20"
+      velocity="1.57" />
   </joint>
   <link
@@ -162,5 +159,5 @@
       </geometry>
       <material
-        name="">
+        name="metal_grey">
         <color
           rgba="1 1 1 1" />
@@ -192,8 +189,6 @@
       lower="-0.0872"
       upper="1.5707"
-      effort="0"
-      velocity="0" />
-    <safety_controller
-      k_velocity="0" />
+      effort="20"
+      velocity="1.57" />
   </joint>
   <link
@@ -222,5 +217,5 @@
       </geometry>
       <material
-        name="">
+        name="metal_grey">
         <color
           rgba="1 1 1 1" />
@@ -252,8 +247,6 @@
       lower="-1.5707"
       upper="0.08726"
-      effort="0"
-      velocity="0" />
-    <safety_controller
-      k_velocity="0" />
+      effort="20"
+      velocity="1.57" />
     <mimic
       joint="magician_joint2"
@@ -267,12 +260,12 @@
         rpy="0 0 0" />
       <mass
-        value="0.001" />
-      <inertia
-        ixx="1.667E-10"
-        ixy="1.667E-10"
-        ixz="1.667E-10"
-        iyy="1.667E-10"
-        iyz="1.667E-10"
-        izz="1.667E-10" />
+        value="0.025" />
+      <inertia
+        ixx="1E-5"
+        ixy="0"
+        ixz="0"
+        iyy="1E-5"
+        iyz="0"
+        izz="1E-5" />
     </inertial>
   </link>
@@ -292,8 +285,6 @@
       lower="-0.2617"
       upper="1.5707"
-      effort="0"
-      velocity="0" />
-    <safety_controller
-      k_velocity="0" />
+      effort="20"
+      velocity="1.57" />
   </joint>
   <link
@@ -322,5 +313,5 @@
       </geometry>
       <material
-        name="">
+        name="metal_grey">
         <color
           rgba="1 1 1 1" />
@@ -352,8 +343,6 @@
       lower="-1.5707"
       upper="0.2617"
-      effort="0"
-      velocity="0" />
-    <safety_controller
-      k_velocity="0" />
+      effort="20"
+      velocity="1.57" />
     <mimic
       joint="magician_joint3"
@@ -413,6 +402,4 @@
     <axis
       xyz="0 0 0" />
-    <safety_controller
-      k_velocity="0" />
   </joint>
   <link
@@ -468,6 +455,4 @@
     <axis
       xyz="0 0 0" />
-    <safety_controller
-      k_velocity="0" />
   </joint>
   <link
@@ -496,5 +481,5 @@
       </geometry>
       <material
-        name="">
+        name="metal_grey">
         <color
           rgba="1 1 1 1" />
@@ -523,6 +508,4 @@
     <axis
       xyz="0 0 0" />
-    <safety_controller
-      k_velocity="0" />
   </joint>
   <link
@@ -551,5 +534,5 @@
       </geometry>
       <material
-        name="">
+        name="metal_grey">
         <color
           rgba="1 1 1 1" />
@@ -578,6 +561,4 @@
     <axis
       xyz="0 0 0" />
-    <safety_controller
-      k_velocity="0" />
   </joint>
 </robot>

Commit message: add magician_moveit_config

File: magician_description/urdf/magician.urdf.xacro (robot description, xacro)
@@ -562,3 +562,17 @@
       xyz="0 0 0" />
   </joint>
+  <link name="magician_end_effctor"/>
+  <joint
+    name="magician_link4_joint1"
+    type="fixed">
+    <origin
+      xyz="-0.05 0 0"
+      rpy="-1.5707963267948966 3.1415926535897932 0" />
+    <parent
+      link="magician_link4" />
+    <child
+      link="magician_end_effctor" />
+    <axis
+      xyz="0 0 0" />
+  </joint>
 </robot>

Commit message: add magician_end_link

File: magician_description/urdf/magician.urdf.xacro (robot description, xacro)
@@ -5,5 +5,4 @@
 <robot
   name="magician" xmlns:xacro="http://www.ros.org/wiki/xacro">
-  <xacro:include filename="$(find magician_description)/urdf/materials.xacro" />
   <xacro:include filename="$(find magician_description)/urdf/magician.gazebo" />
   <xacro:include filename="$(find magician_description)/urdf/magician_transmission.xacro" />
@@ -159,7 +158,7 @@
       </geometry>
       <material
-        name="metal_grey">
-        <color
-          rgba="1 1 1 1" />
+        name="">
+        <color
+          rgba="0.501960784313725 0.501960784313725 0.501960784313725 1" />
       </material>
     </visual>
@@ -217,7 +216,7 @@
       </geometry>
       <material
-        name="metal_grey">
-        <color
-          rgba="1 1 1 1" />
+        name="">
+        <color
+          rgba="0.501960784313725 0.501960784313725 0.501960784313725 1" />
       </material>
     </visual>
@@ -313,7 +312,7 @@
       </geometry>
       <material
-        name="metal_grey">
-        <color
-          rgba="1 1 1 1" />
+        name="">
+        <color
+          rgba="0.501960784313725 0.501960784313725 0.501960784313725 1" />
       </material>
     </visual>
@@ -377,5 +376,5 @@
         name="">
         <color
-          rgba="1 1 1 1" />
+          rgba="0.501960784313725 0.501960784313725 0.501960784313725 1" />
       </material>
     </visual>
@@ -430,5 +429,5 @@
         name="">
         <color
-          rgba="1 1 1 1" />
+          rgba="0.501960784313725 0.501960784313725 0.501960784313725 1" />
       </material>
     </visual>
@@ -481,7 +480,7 @@
       </geometry>
       <material
-        name="metal_grey">
-        <color
-          rgba="1 1 1 1" />
+        name="">
+        <color
+          rgba="0.501960784313725 0.501960784313725 0.501960784313725 1" />
       </material>
     </visual>
@@ -534,7 +533,7 @@
       </geometry>
       <material
-        name="metal_grey">
-        <color
-          rgba="1 1 1 1" />
+        name="">
+        <color
+          rgba="0.501960784313725 0.501960784313725 0.501960784313725 1" />
       </material>
     </visual>
@@ -562,13 +561,27 @@
       xyz="0 0 0" />
   </joint>
+  <link name="magician_end_link"/>
+  <joint
+    name="magician_link4_joint1"
+    type="fixed">
+    <origin
+      xyz="0 0 0"
+      rpy="-1.5707963267948966 3.1415926535897932 0" />
+    <parent
+      link="magician_link4" />
+    <child
+      link="magician_end_link" />
+    <axis
+      xyz="0 0 0" />
+  </joint>
   <link name="magician_end_effctor"/>
   <joint
-    name="magician_link4_joint1"
-    type="fixed">
-    <origin
-      xyz="-0.05 0 0"
-      rpy="-1.5707963267948966 3.1415926535897932 0" />
-    <parent
-      link="magician_link4" />
+    name="magician_end_link_joint1"
+    type="fixed">
+    <origin
+      xyz="0.05 0 0"
+      rpy="0 0 0" />
+    <parent
+      link="magician_end_link" />
     <child
       link="magician_end_effctor" />

Commit message: add a new joint magician_fake_joint3

File: magician_description/urdf/magician.urdf.xacro (robot description, xacro)
@@ -7,4 +7,10 @@
   <xacro:include filename="$(find magician_description)/urdf/magician.gazebo" />
   <xacro:include filename="$(find magician_description)/urdf/magician_transmission.xacro" />
+  <xacro:property name="joint1_lower" value="-2.1816"/>
+  <xacro:property name="joint1_upper" value="2.1816"/>
+  <xacro:property name="joint2_lower" value="-0.087"/>
+  <xacro:property name="joint2_upper" value="0.872"/>
+  <xacro:property name="joint3_lower" value="-0.087"/>
+  <xacro:property name="joint3_upper" value="1.134"/>
   <link name="world"/>
   <link name="magician_origin"/>
@@ -128,6 +134,6 @@
       xyz="0 0 1" />
     <limit
-      lower="-2.1816"
-      upper="2.1816"
+      lower="${joint1_lower}"
+      upper="${joint1_upper}"
       effort="20"
       velocity="1.57" />
@@ -186,6 +192,6 @@
       xyz="0 0 1" />
     <limit
-      lower="-0.0872"
-      upper="1.5707"
+      lower="${joint2_lower}"
+      upper="${joint2_upper}"
       effort="20"
       velocity="1.57" />
@@ -244,6 +250,6 @@
       xyz="0 0 -1" />
     <limit
-      lower="-1.5707"
-      upper="0.08726"
+      lower="${-1*joint2_upper}"
+      upper="${-1*joint2_lower}"
       effort="20"
       velocity="1.57" />
@@ -282,6 +288,6 @@
       xyz="0 0 -1" />
     <limit
-      lower="-0.2617"
-      upper="1.5707"
+      lower="${joint3_lower}"
+      upper="${joint3_upper}"
       effort="20"
       velocity="1.57" />
@@ -340,6 +346,6 @@
       xyz="0 0 1" />
     <limit
-      lower="-1.5707"
-      upper="0.2617"
+      lower="${-1*joint3_upper}"
+      upper="${-1*joint3_lower}"
       effort="20"
       velocity="1.57" />
@@ -561,4 +567,27 @@
       xyz="0 0 0" />
   </joint>
+  <link name="magician_end_turnplate"/>
+  <joint
+    name="magician_fake_joint3"
+    type="revolute">
+    <origin
+      xyz="0 0 0"
+      rpy="-1.5707963267948966 3.1415926535897932 0" />
+    <parent
+      link="magician_link4" />
+    <child
+      link="magician_end_turnplate" />
+    <axis
+      xyz="0 0 1" />
+    <limit
+      lower="${-1*joint1_upper}"
+      upper="${-1*joint1_lower}"
+      effort="20"
+      velocity="1.57" />
+    <mimic
+      joint="magician_joint1"
+      multiplier="-1"
+      offset="0"/>
+  </joint>
   <link name="magician_end_link"/>
   <joint
@@ -567,7 +596,7 @@
     <origin
       xyz="0 0 0"
-      rpy="-1.5707963267948966 3.1415926535897932 0" />
-    <parent
-      link="magician_link4" />
+      rpy="0 0 0" />
+    <parent
+      link="magician_end_turnplate" />
     <child
       link="magician_end_link" />

Commit message: add magician_kinematics

File: magician_description/urdf/magician.urdf.xacro (robot description, xacro)
@@ -355,4 +355,16 @@
       offset="0"/>
   </joint>
+  <link name="magician_arm_end"/>
+  <joint
+    name="magician_link4_joint1"
+    type="fixed">
+    <origin
+      xyz="0 0 0"
+      rpy="-1.5707963267948966 3.1415926535897932 0" />
+    <parent
+      link="magician_link4" />
+    <child
+      link="magician_arm_end" />
+  </joint>
   <link
     name="magician_link3_surface">
@@ -573,7 +585,7 @@
     <origin
       xyz="0 0 0"
-      rpy="-1.5707963267948966 3.1415926535897932 0" />
-    <parent
-      link="magician_link4" />
+      rpy="0 0 0" />
+    <parent
+      link="magician_arm_end" />
     <child
       link="magician_end_turnplate" />
@@ -592,5 +604,5 @@
   <link name="magician_end_link"/>
   <joint
-    name="magician_link4_joint1"
+    name="magician_end_turnplate_joint1"
     type="fixed">
     <origin
@@ -609,5 +621,5 @@
     type="fixed">
     <origin
-      xyz="0.05 0 0"
+      xyz="0 0 0"
       rpy="0 0 0" />
     <parent

Commit message: set new joint limits

File: magician_description/urdf/magician.urdf.xacro (robot description, xacro)
@@ -9,8 +9,8 @@
   <xacro:property name="joint1_lower" value="-2.1816"/>
   <xacro:property name="joint1_upper" value="2.1816"/>
-  <xacro:property name="joint2_lower" value="-0.087"/>
-  <xacro:property name="joint2_upper" value="0.872"/>
-  <xacro:property name="joint3_lower" value="-0.087"/>
-  <xacro:property name="joint3_upper" value="1.134"/>
+  <xacro:property name="joint2_lower" value="0.35"/>
+  <xacro:property name="joint2_upper" value="1.57"/>
+  <xacro:property name="joint3_lower" value="0.62"/>
+  <xacro:property name="joint3_upper" value="1.57"/>
   <link name="world"/>
   <link name="magician_origin"/>
@@ -136,5 +136,5 @@
       lower="${joint1_lower}"
       upper="${joint1_upper}"
-      effort="20"
+      effort="6"
       velocity="1.57" />
   </joint>
@@ -194,5 +194,5 @@
       lower="${joint2_lower}"
       upper="${joint2_upper}"
-      effort="20"
+      effort="6"
       velocity="1.57" />
   </joint>
@@ -252,5 +252,5 @@
       lower="${-1*joint2_upper}"
       upper="${-1*joint2_lower}"
-      effort="20"
+      effort="6"
       velocity="1.57" />
     <mimic
@@ -267,10 +267,10 @@
         value="0.025" />
       <inertia
-        ixx="1E-5"
+        ixx="2.5E-4"
         ixy="0"
         ixz="0"
-        iyy="1E-5"
+        iyy="2.5E-4"
         iyz="0"
-        izz="1E-5" />
+        izz="2.5E-4" />
     </inertial>
   </link>
@@ -290,5 +290,5 @@
       lower="${joint3_lower}"
       upper="${joint3_upper}"
-      effort="20"
+      effort="6"
       velocity="1.57" />
   </joint>
@@ -348,5 +348,5 @@
       lower="${-1*joint3_upper}"
       upper="${-1*joint3_lower}"
-      effort="20"
+      effort="6"
       velocity="1.57" />
     <mimic
@@ -595,5 +595,5 @@
       lower="${-1*joint1_upper}"
       upper="${-1*joint1_lower}"
-      effort="20"
+      effort="6"
       velocity="1.57" />
     <mimic
